File: CC1101_Module.kicad_pcb (KiCad board)
At the start: 2 copper layers, 19.9 x 16.7 mm, 27 parts, among them J1 Conn, J10 Conn, J4 Conn, J5 Conn, J6 Conn, J7 Conn, J8 Conn, J9 Conn, U1 CC1101RTK, Y1 Resonator_Small

Commit message: update kicad
Other:
- net class Default removed
